File: VCO.sch (KiCad schematic (older format))
At the start: 76 parts, among them J1 Conn_01x05_Male, J10 FM, J12 PW, J13 saw, J14 sq, J3 V/oct, J4 Conn_01x05_Male, J5 Conn_01x05_Male, J6 Conn_01x05_Male, J8 Conn_01x05_Male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

Commit message: Add led's. Issue #8 close
Parts:
- added D1: LED_SQ, footprint:led_0603, symbol uRack:LED
- added D2: LED_SAW, footprint:led_0603, symbol uRack:LED
- added R45, R46: 100R, footprint:r0603, symbol uRack:R
Connections:
- wire segments 266 -> 276
Other:
- moved on the sheet: J13, R40, R41, R42, R43

Commit message: Change position power connector add mounting hole 3.2 mm diametr Issue #7 closed
Parts:
- removed J1, J4, J5, J6, J8, J9: Conn_01x05_Male, footprint:pls1x05, symbol uRack:Conn_01x05_Male
- added J1, J4, J8, J9: Conn_01x04_Male, footprint:pls1x04, symbol uRack:Conn_01x04_Male
- added J5, J6: Conn_01x03_Male, footprint:pls1x03, symbol uRack:Conn_01x03_Male
Connections:
- wire segments 276 -> 260
Changed lines of the file:
@@
 Wire Wire Line
 	6450 7100 6450 7250
-$Comp
-L uRack:Conn_01x05_Male J4
-U 1 1 5C943416
-P 10400 1500
-F 0 "J4" H 10373 1430 50  0000 R CNN
-F 1 "Conn_01x05_Male" H 10373 1521 50  0000 R CNN
-F 2 "footprint:pls1x05" H 10400 1500 50  0001 C CNN
-F 3 "" H 10400 1500 50  0001 C CNN
-	1    10400 1500
-	-1   0    0    1
-$EndComp
-$Comp
-L uRack:Conn_01x05_Male J1
-U 1 1 5C943702
-P 10400 900
-F 0 "J1" H 10373 830 50  0000 R CNN
-F 1 "Conn_01x05_Male" H 10373 921 50  0000 R CNN
-F 2 "footprint:pls1x05" H 10400 900 50  0001 C CNN
-F 3 "" H 10400 900 50  0001 C CNN
-	1    10400 900
-	-1   0    0    1
-$EndComp
-$Comp
-L uRack:Conn_01x05_Male J6
-U 1 1 5C94397B
-P 10450 2550
-F 0 "J6" H 10423 2480 50  0000 R CNN
-F 1 "Conn_01x05_Male" H 10423 2571 50  0000 R CNN
-F 2 "footprint:pls1x05" H 10450 2550 50  0001 C CNN
-F 3 "" H 10450 2550 50  0001 C CNN
-	1    10450 2550
-	-1   0    0    1
-$EndComp
-$Comp
-L uRack:Conn_01x05_Male J5
-U 1 1 5C943AE1
-P 10450 2050
-F 0 "J5" H 10423 1980 50  0000 R CNN
-F 1 "Conn_01x05_Male" H 10423 2071 50  0000 R CNN
-F 2 "footprint:pls1x05" H 10450 2050 50  0001 C CNN
-F 3 "" H 10450 2050 50  0001 C CNN
-	1    10450 2050
-	-1   0    0    1
-$EndComp
-$Comp
-L uRack:Conn_01x05_Male J8
-U 1 1 5C945263
-P 10600 3450
-F 0 "J8" H 10573 3380 50  0000 R CNN
-F 1 "Conn_01x05_Male" V 10400 3400 50  0000 R CNN
-F 2 "footprint:pls1x05" H 10600 3450 50  0001 C CNN
-F 3 "" H 10600 3450 50  0001 C CNN
-	1    10600 3450
-	-1   0    0    1
-$EndComp
-$Comp
-L uRack:Conn_01x05_Male J9
-U 1 1 5C945356
-P 10600 3950
-F 0 "J9" H 10573 3880 50  0000 R CNN
-F 1 "Conn_01x05_Male" V 10400 4100 50  0000 R CNN
-F 2 "footprint:pls1x05" H 10600 3950 50  0001 C CNN
-F 3 "" H 10600 3950 50  0001 C CNN
-	1    10600 3950
-	-1   0    0    1
-$EndComp
-Wire Wire Line
-	10250 3250 10400 3250
-Wire Wire Line
-	10400 3350 10250 3350
-Connection ~ 10250 3350
-Wire Wire Line
-	10250 3350 10250 3250
-Wire Wire Line
-	10400 3450 10250 3450
-Connection ~ 10250 3450
-Wire Wire Line
-	10250 3450 10250 3350
-Wire Wire Line
-	10400 3550 10250 3550
-Connection ~ 10250 3550
-Wire Wire Line
-	10250 3550 10250 3450
-Wire Wire Line
-	10400 3650 10250 3650
-Connection ~ 10250 3650
-Wire Wire Line
-	10250 3650 10250 3550
-Wire Wire Line
-	10400 3750 10250 3750
-Connection ~ 10250 3750
-Wire Wire Line
-	10250 3750 10250 3650
-Wire Wire Line
-	10400 3850 10250 3850
-Connection ~ 10250 3850
-Wire Wire Line
-	10250 3850 10250 3750
-Wire Wire Line
-	10400 3950 10250 3950
-Connection ~ 10250 3950
-Wire Wire Line
-	10250 3950 10250 3850
-Wire Wire Line
-	10400 4050 10250 4050
-Connection ~ 10250 4050
-Wire Wire Line
-	10250 4050 10250 3950
-Wire Wire Line
-	10400 4150 10250 4150
-Wire Wire Line
-	10250 4150 10250 4050
-Wire Wire Line
-	10200 1850 10250 1850
-Wire Wire Line
-	10250 1950 10200 1950
-Connection ~ 10200 1950
-Wire Wire Line
-	10200 1950 10200 1850
-Wire Wire Line
-	10250 2750 10200 2750
-Connection ~ 10200 2750
-Wire Wire Line
-	10200 2750 10200 2650
-Wire Wire Line
-	10250 2650 10200 2650
-Connection ~ 10200 2650
-Wire Wire Line
-	10200 2650 10200 2550
-Wire Wire Line
-	10250 2550 10200 2550
-Connection ~ 10200 2550
-Wire Wire Line
-	10200 2550 10200 2450
-Wire Wire Line
-	10250 2450 10200 2450
-Connection ~ 10200 2450
-Wire Wire Line
-	10200 2450 10200 2350
-Wire Wire Line
-	10250 2350 10200 2350
-Connection ~ 10200 2350
-Wire Wire Line
-	10200 2350 10200 2250
-Wire Wire Line
-	10250 2250 10200 2250
-Connection ~ 10200 2250
-Wire Wire Line
-	10200 2250 10200 2150
-Wire Wire Line
-	10250 2150 10200 2150
-Connection ~ 10200 2150
-Wire Wire Line
-	10200 2150 10200 2050
-Wire Wire Line
-	10250 2050 10200 2050
-Connection ~ 10200 2050
-Wire Wire Line
-	10200 2050 10200 1950
-Wire Wire Line
-	10200 1700 10150 1700
-Wire Wire Line
-	10150 1700 10150 1600
+Wire Wire Line
+	10150 2850 10300 2850
+Wire Wire Line
+	10300 2950 10150 2950
+Connection ~ 10150 2950
+Wire Wire Line
+	10150 2950 10150 2850
+Wire Wire Line
+	10300 3050 10150 3050
+Connection ~ 10150 3050
+Wire Wire Line
+	10150 3050 10150 2950
+Wire Wire Line
+	10300 3150 10150 3150
+Connection ~ 10150 3150
+Wire Wire Line
+	10150 3150 10150 3050
+Wire Wire Line
+	10300 3350 10150 3350
+Connection ~ 10150 3350
+Wire Wire Line
+	10300 3450 10150 3450
+Connection ~ 10150 3450
+Wire Wire Line
+	10150 3450 10150 3350
+Wire Wire Line
+	10300 3550 10150 3550
+Connection ~ 10150 3550
+Wire Wire Line
+	10150 3550 10150 3450
+Wire Wire Line
+	10300 3650 10150 3650
+Wire Wire Line
+	10150 3650 10150 3550
+Wire Wire Line
+	10150 1850 10200 1850
+Wire Wire Line
+	10200 1950 10150 1950
+Connection ~ 10150 1950
+Wire Wire Line
+	10150 1950 10150 1850
+Wire Wire Line
+	10200 2350 10150 2350
+Wire Wire Line
+	10150 2350 10150 2250
+Wire Wire Line
+	10200 2250 10150 2250
+Connection ~ 10150 2250
+Wire Wire Line
+	10150 2250 10150 2150
+Wire Wire Line
+	10200 2150 10150 2150
+Connection ~ 10150 2150
+Wire Wire Line
+	10150 2150 10150 2050
+Wire Wire Line
+	10200 2050 10150 2050
+Connection ~ 10150 2050
+Wire Wire Line
+	10150 2050 10150 1950
 Wire Wire Line
 	10150 700  10200 700
@@
 	10150 1000 10150 900
 Wire Wire Line
-	10200 1100 10150 1100
-Connection ~ 10150 1100
-Wire Wire Line
-	10150 1100 10150 1000
-Wire Wire Line
 	10200 1300 10150 1300
 Connection ~ 10150 1300
@@
 Wire Wire Line
 	10200 1600 10150 1600
-Connection ~ 10150 1600
 $Comp
 L uRack:R_POT RV2
@@
 	4350 3750 4350 3000
 Connection ~ 4100 3750
-Connection ~ 10250 3250
+Connection ~ 10150 2850
 Text Label 8950 5450 0    50   ~ 0
 saw
@@
 Wire Wire Line
 	6200 4700 6200 5400
-Wire Wire Line
-	10200 2750 10200 2900
-Wire Wire Line
-	10150 1100 10150 1300
 $Comp
 L uRack:BC847BS Q1
@@
 L uRack:-9V #PWR0102
 U 1 1 5FA1EE51
-P 10250 3250
-F 0 "#PWR0102" H 10250 3125 50  0001 C CNN
-F 1 "-9V" V 10265 3378 50  0000 L CNN
-F 2 "" H 10250 3250 50  0001 C CNN
-F 3 "" H 10250 3250 50  0001 C CNN
-	1    10250 3250
+P 10150 2850
+F 0 "#PWR0102" H 10150 2725 50  0001 C CNN
+F 1 "-9V" V 10165 2978 50  0000 L CNN
+F 2 "" H 10150 2850 50  0001 C CNN
+F 3 "" H 10150 2850 50  0001 C CNN
+	1    10150 2850
 	0    -1   -1   0
 $EndComp
@@
 L uRack:GNDREF #PWR0131
 U 1 1 5FC1CEB4
-P 10200 2900
-F 0 "#PWR0131" H 10200 2650 50  0001 C CNN
-F 1 "GNDREF" H 10205 2727 50  0000 C CNN
-F 2 "" H 10200 2900 50  0001 C CNN
-F 3 "" H 10200 2900 50  0001 C CNN
-	1    10200 2900
+P 10150 2450
+F 0 "#PWR0131" H 10150 2200 50  0001 C CNN
+F 1 "GNDREF" H 10155 2277 50  0000 C CNN
+F 2 "" H 10150 2450 50  0001 C CNN
+F 3 "" H 10150 2450 50  0001 C CNN
+	1    10150 2450
 	1    0    0    -1
 $EndComp
@@
 Wire Wire Line
 	9700 5550 9950 5550
+$Comp
+L uRack:Conn_01x04_Male J1
+U 1 1 5FA79323
+P 10400 900
+F 0 "J1" H 10372 782 50  0000 R CNN
+F 1 "Conn_01x04_Male" H 10372 873 50  0000 R CNN
+F 2 "footprint:pls1x04" H 10400 900 50  0001 C CNN
+F 3 "" H 10400 900 50  0001 C CNN
+	1    10400 900
+	-1   0    0    1
+$EndComp
+$Comp
+L uRack:Conn_01x04_Male J4
+U 1 1 5FA79F08
+P 10400 1500
+F 0 "J4" H 10372 1382 50  0000 R CNN
+F 1 "Conn_01x04_Male" H 10372 1473 50  0000 R CNN
+F 2 "footprint:pls1x04" H 10400 1500 50  0001 C CNN
+F 3 "" H 10400 1500 50  0001 C CNN
+	1    10400 1500
+	-1   0    0    1
+$EndComp
+Wire Wire Line
+	10150 1000 10150 1300
+$Comp
+L uRack:Conn_01x03_Male J5
+U 1 1 5FA8330B
+P 10400 1950
+F 0 "J5" H 10372 1882 50  0000 R CNN
+F 1 "Conn_01x03_Male" H 10372 1973 50  0000 R CNN
+F 2 "footprint:pls1x03" H 10400 1950 50  0001 C CNN
+F 3 "" H 10400 1950 50  0001 C CNN
+	1    10400 1950
+	-1   0    0    1
+$EndComp
+$Comp
+L uRack:Conn_01x03_Male J6
+U 1 1 5FA83B98
+P 10400 2250
+F 0 "J6" H 10372 2182 50  0000 R CNN
+F 1 "Conn_01x03_Male" H 10372 2273 50  0000 R CNN
+F 2 "footprint:pls1x03" H 10400 2250 50  0001 C CNN
+F 3 "" H 10400 2250 50  0001 C CNN
+	1    10400 2250
+	-1   0    0    1
+$EndComp
+Wire Wire Line
+	10150 2450 10150 2350
+Connection ~ 10150 2350
+$Comp
+L uRack:Conn_01x04_Male J8
+U 1 1 5FAC1065
+P 10500 3050
+F 0 "J8" H 10472 2932 50  0000 R CNN
+F 1 "Conn_01x04_Male" H 10472 3023 50  0000 R CNN
+F 2 "footprint:pls1x04" H 10500 3050 50  0001 C CNN
+F 3 "" H 10500 3050 50  0001 C CNN
+	1    10500 3050
+	-1   0    0    1
+$EndComp
+$Comp
+L uRack:Conn_01x04_Male J9
+U 1 1 5FAC1B61
+P 10500 3550
+F 0 "J9" H 10472 3432 50  0000 R CNN
+F 1 "Conn_01x04_Male" H 10472 3523 50  0000 R CNN
+F 2 "footprint:pls1x04" H 10500 3550 50  0001 C CNN
+F 3 "" H 10500 3550 50  0001 C CNN
+	1    10500 3550
+	-1   0    0    1
+$EndComp
+Wire Wire Line
+	10150 3150 10150 3350
 $EndSCHEMATC

Commit message: Change current led's resistor 100R to 1K
Parts:
- R45, R46: value 100R -> 1K
Changed lines of the file:
@@
 P 8200 5250
 F 0 "R45" H 8350 5200 50  0000 C CNN
-F 1 "100R" H 8350 5300 50  0000 C CNN
+F 1 "1K" H 8350 5300 50  0000 C CNN
 F 2 "footprint:r0603" V 8130 5250 50  0001 C CNN
 F 3 "~" H 8200 5250 50  0001 C CNN
@@
 P 9550 5550
 F 0 "R46" V 9500 5350 50  0000 C CNN
-F 1 "100R" V 9600 5750 50  0000 C CNN
+F 1 "1K" V 9600 5750 50  0000 C CNN
 F 2 "footprint:r0603" V 9480 5550 50  0001 C CNN
 F 3 "~" H 9550 5550 50  0001 C CNN

Commit message: add power protection change power connector
Parts:
- removed J5, J6: Conn_01x03_Male, footprint:pls1x03, symbol uRack:Conn_01x03_Male
- removed J8, J9: Conn_01x04_Male, footprint:pls1x04, symbol uRack:Conn_01x04_Male
- added J5, J6: PLS2x4, footprint:pls2x04, symbol uRack:PLS2x4
- added Q2: IRLML5203, footprint:SOT-23, symbol uRack:IRLML5203
- C10, C7, C8, C9: footprint Capacitor_SMD:C_0603_1608Metric_Pad1.05x0.95mm_HandSolder -> footprint:c0603
Connections:
- wire segments 260 -> 254
Other:
- moved on the sheet: C1, C10, C2, C3, C4, C5, C6, C7, C8, C9, J10, J12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
